Commit message: Add files via upload

File: urdf/accessories/lidar_volta.urdf.xacro (robot description, xacro)
@@ -25,5 +25,5 @@
 -->
 <robot name="volta_robot" xmlns:xacro="https://ros.org/wiki/xacro">
-  <xacro:macro name="lidar" params="frame:=lidar topic:=scan_filtered sample_size:=271 update_rate:=50
+  <xacro:macro name="lidar" params="frame:=lidar topic:=scan sample_size:=271 update_rate:=50
                  min_angle:=-1.57 max_angle:=1.57 min_range:=0.5 max_range:=10.0 rplidar_a3_enabled:=true hokuyo_ust_10lx_enabled:=false robot_namespace:=/">
       <xacro:if value="${rplidar_a3_enabled}">

File: urdf/volta.urdf.xacro (robot description, xacro)
@@ -43,10 +43,10 @@
     <xacro:macro name="volta_robot">
         <!-- Footprint -->
-        <link name="footprint"/>
+        <link name="base_footprint"/>
         <!-- Joint from footprint to base link(chassis) -->
         <joint name="base_footprint_joint" type="fixed">
             <origin xyz="0 0 ${base_underside_h}" rpy="0 0 0" />
             <parent link="base_link" />
-            <child link="footprint" />
+            <child link="base_footprint" />
         </joint>
         <!-- Chassis a.k.a base_link -->
